File: pidControllerResources/pidControllerRev8.brd (EAGLE design)
At the start: 88.9 x 101.6 mm, 79 parts, among them IC1 TLC274P, IC2 TLC274P, IC3 TLC274P, IC4 TLC274P, J4 INPUT, Q1 2N7000, T1 2N3906, T2 2N3906

Commit message: Update the file name
Parts:
- added S3: CLEAR, SparkFun-Switches:TACTILE_SWITCH_SMD_5.2MM
Connections:
- net I_TERM: now also S3.1
- net N$4: now also S3.3
Routing:
- net N$4: track 10.8 -> 19.2 mm
- net I_TERM: track 96.2 -> 98.0 mm
Changed lines of the file:
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@@
 <attribute name="VALUE" x="65.278" y="95.504" size="0.6096" layer="27" font="vector" ratio="20"/>
+</element>
+<element name="S3" library="SparkFun-Switches" package="TACTILE_SWITCH_SMD_5.2MM" value="CLEAR" x="50.8" y="54.356" smashed="yes">
+<attribute name="NAME" x="50.8" y="54.737" size="1.016" layer="25" font="vector" rot="R180" align="bottom-center"/>
+<attribute name="PROD_ID" value="SWCH-08247" x="50.8" y="54.356" size="1.016" layer="27" display="off"/>
+<attribute name="SF_SKU" value="COM-08720" x="50.8" y="54.356" size="1.016" layer="27" display="off"/>
+<attribute name="VALUE" x="45.212" y="54.737" size="1.016" layer="27" font="vector" align="top-center"/>
 </element>
 </elements>
@@
 <contactref element="C4" pad="2"/>
 <contactref element="IC1" pad="1"/>
-<wire x1="48.768" y1="73.152" x2="48.768" y2="79.248" width="0.4064" layer="1"/>
+<wire x1="48.768" y1="73.152" x2="48.768" y2="80.4418" width="0.4064" layer="1"/>
 <via x="48.768" y="73.152" extent="1-16" drill="0.35"/>
-<wire x1="48.768" y1="79.248" x2="48.768" y2="79.9338" width="0.4064" layer="1"/>
 <wire x1="23.0378" y1="42.5958" x2="26.1499875" y2="42.5958" width="0.4064" layer="1"/>
 <wire x1="26.1499875" y1="42.5958" x2="27.6739875" y2="44.1198" width="0.4064" layer="1"/>
@@
 <via x="46.228" y="68.072" extent="1-16" drill="0.35"/>
 <wire x1="48.768" y1="73.152" x2="46.228" y2="70.612" width="0.4064" layer="16"/>
-<wire x1="46.228" y1="51.308" x2="46.228" y2="59.944" width="0.4064" layer="1"/>
+<wire x1="46.228" y1="57.404" x2="46.228" y2="59.944" width="0.4064" layer="1"/>
 <wire x1="27.6739875" y1="44.1198" x2="40.0558" y2="44.1198" width="0.4064" layer="1"/>
 <via x="41.148" y="45.212" extent="1-16" drill="0.35"/>
@@
 <wire x1="33.3502" y1="92.964" x2="36.2458" y2="92.964" width="0.4064" layer="1"/>
 <wire x1="36.2458" y1="92.964" x2="48.768" y2="80.4418" width="0.4064" layer="1"/>
-<wire x1="48.768" y1="80.4418" x2="48.768" y2="79.9338" width="0.4064" layer="1"/>
+<contactref element="S3" pad="1"/>
+<wire x1="48.006" y1="56.261" x2="47.371" y2="56.261" width="0.4064" layer="1"/>
+<wire x1="47.371" y1="56.261" x2="46.228" y2="57.404" width="0.4064" layer="1"/>
+<wire x1="48.006" y1="56.261" x2="46.228" y2="54.483" width="0.4064" layer="1"/>
+<wire x1="46.228" y1="54.483" x2="46.228" y2="51.308" width="0.4064" layer="1"/>
 </signal>
 <signal name="N$6">
@@
 <wire x1="58.674" y1="59.944" x2="57.782" y2="59.052" width="0.4064" layer="1"/>
 <wire x1="57.782" y1="59.052" x2="52.324" y2="59.052" width="0.4064" layer="1"/>
+<contactref element="S3" pad="3"/>
+<wire x1="48.006" y1="52.451" x2="52.324" y2="56.769" width="0.4064" layer="1"/>
+<wire x1="52.324" y1="56.769" x2="52.324" y2="59.052" width="0.4064" layer="1"/>
 </signal>
 <signal name="N$18">
