File: pidControllerResources/pidControllerRev8.sch (EAGLE design)
At the start: 79 parts, among them IC1 TLC274P, IC2 TLC274P, IC3 TLC274P, IC4 TLC274P, J4 INPUT, Q1 2N7000, T1 2N3906, T2 2N3906

Commit message: Update the file name
Parts:
- added S3: CLEAR, SparkFun-Switches:MOMENTARY-SWITCH-SPST-SMD-5.2MM
Connections:
- net I_TERM: now also S3.1
- net N$4: now also S3.2
Changed lines of the file:
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@@
 <part name="PWM" library="SparkFun-Connectors" deviceset="CONN_02" device="LOCK"/>
 <part name="OUT" library="SparkFun-Connectors" deviceset="CONN_02" device="LOCK"/>
+<part name="S3" library="SparkFun-Switches" deviceset="MOMENTARY-SWITCH-SPST" device="-SMD-5.2MM" value="CLEAR"/>
 </parts>
 <sheets>
@@
 <attribute name="NAME" x="289.56" y="264.668" size="1.778" layer="95" font="vector"/>
 </instance>
+<instance part="S3" gate="G$1" x="101.6" y="45.72" smashed="yes" rot="R180">
+<attribute name="NAME" x="101.6" y="44.196" size="1.778" layer="95" font="vector" rot="R180" align="bottom-center"/>
+<attribute name="VALUE" x="101.6" y="46.228" size="1.778" layer="96" font="vector" rot="R180" align="top-center"/>
+</instance>
 </instances>
 <busses>
@@
 <junction x="121.92" y="66.04"/>
 <label x="127" y="66.04" size="1.778" layer="95" xref="yes"/>
+<pinref part="S3" gate="G$1" pin="1"/>
+<wire x1="106.68" y1="45.72" x2="121.92" y2="45.72" width="0.1524" layer="91"/>
+<wire x1="121.92" y1="45.72" x2="121.92" y2="53.34" width="0.1524" layer="91"/>
+<junction x="121.92" y="53.34"/>
 </segment>
 </net>
@@
 <wire x1="91.44" y1="53.34" x2="91.44" y2="63.5" width="0.1524" layer="91"/>
 <junction x="91.44" y="63.5"/>
-</segment>
-</net>
+<pinref part="S3" gate="G$1" pin="2"/>
+<wire x1="96.52" y1="45.72" x2="91.44" y2="45.72" width="0.1524" layer="91"/>
+<wire x1="91.44" y1="45.72" x2="91.44" y2="53.34" width="0.1524" layer="91"/>
+<junction x="91.44" y="53.34"/>
+</segment>
+</net>
