File: curveTracerResources/curveTracerRev5.sch (EAGLE design)
At the start: 60 parts, among them IC1 555, IC2 TLC274P, Q1 2N7000, Q2 2N7000, Q3 2N7000, Q4 2N3906, Q5 2N3906, Q6 2N7000

Commit message: update to rev 5 - the latest
Parts:
- removed PWR: (no value), con-jack:JACK-PLUG0
Connections:
- net GND_IN: no longer PWR.1, PWR.2
- net N$1: no longer PWR.3
Other:
- moved on the sheet: GNDIN
