File: audioBoardResources/audioRev5.sch (EAGLE design)
At the start: 60 parts, among them IC1 MCP604P, IC2 78L05Z, J9 AUDIO_JACK_3.5MM, Q1 FQP27P06, T1 TIP 31, T2 TIP 32, T3 2N3904, T4 2N3904

Commit message: update audioBoard to correct and latest version
Parts:
- removed J1: (no value), con-jack:JACK-PLUG0
- R16: value 1k -> 33k
Connections:
- removed net DRAIN: J1.3, Q1.D, VIN.1, VIN.2
- new net VIN: Q1.D, VIN.1, VIN.2
- net GND: no longer J1.1, J1.2
